File: hw/differential_probe/amplifiers.kicad_sch (KiCad schematic)
At the start: 31 parts, among them U3 THS4631D, U4 THS4631D, U5 THS4631D

Commit message: initial routing
Parts:
- added R55: 0R, Resistor_SMD:R_0402_1005Metric_Pad0.72x0.64mm_HandSolder, symbol Device:R
- C56: renamed from C35; value 3.3u -> 10u; footprint (none) -> Capacitor_SMD:C_1206_3216Metric; LCSC (none) -> C13585
- C57: renamed from C36; footprint (none) -> Capacitor_SMD:C_0402_1005Metric; LCSC (none) -> C307331
- C58: renamed from C37; footprint (none) -> Capacitor_SMD:C_0402_1005Metric; LCSC (none) -> C307331
- C59: renamed from C34; value 0.25p -> 0.3p; footprint (none) -> Capacitor_SMD:C_0402_1005Metric_Pad0.74x0.62mm_HandSolder; MFR PART # (none) -> GJM1555C1HR30WB01D
- C60: renamed from C43; footprint (none) -> Capacitor_SMD:C_0402_1005Metric_Pad0.74x0.62mm_HandSolder; MFR PART # (none) -> GJM1555C1HR80WB01D
- C61: renamed from C38; value 3.3u -> 10u; footprint (none) -> Capacitor_SMD:C_1206_3216Metric; LCSC (none) -> C13585
- C62: renamed from C49; value 3.3u -> 10u; footprint (none) -> Capacitor_SMD:C_1206_3216Metric; LCSC (none) -> C13585
- C63: renamed from C50; footprint (none) -> Capacitor_SMD:C_0402_1005Metric; LCSC (none) -> C307331
- C64: renamed from C41; value 3.3u -> 10u; footprint (none) -> Capacitor_SMD:C_1206_3216Metric; LCSC (none) -> C13585
- C65: renamed from C42; footprint (none) -> Capacitor_SMD:C_0402_1005Metric; LCSC (none) -> C307331
- C66: renamed from C51; footprint (none) -> Capacitor_SMD:C_0402_1005Metric; LCSC (none) -> C307331
- C67: renamed from C48; value 0.5p -> 0.3p; footprint (none) -> Capacitor_SMD:C_0402_1005Metric_Pad0.74x0.62mm_HandSolder; MFR PART # (none) -> GJM1555C1HR30WB01D
- C68: renamed from C52; value 3.3u -> 10u; footprint (none) -> Capacitor_SMD:C_1206_3216Metric; LCSC (none) -> C13585
- C69: renamed from C44; footprint (none) -> Capacitor_SMD:C_0402_1005Metric; LCSC (none) -> C307331
- C70: renamed from C40; value 0.25p -> 0.3p; footprint (none) -> Capacitor_SMD:C_0402_1005Metric_Pad0.74x0.62mm_HandSolder; MFR PART # (none) -> GJM1555C1HR30WB01D
- C71: renamed from C47; footprint (none) -> Capacitor_SMD:C_0402_1005Metric_Pad0.74x0.62mm_HandSolder; MFR PART # (none) -> GJM1555C1HR80WB01D
- C72: renamed from C45; value 3.3u -> 10u; footprint (none) -> Capacitor_SMD:C_1206_3216Metric; LCSC (none) -> C13585
- L2: renamed from L3; value 33n -> 47n; footprint (none) -> Inductor_SMD:L_0402_1005Metric_Pad0.77x0.64mm_HandSolder; MFR PART # (none) -> LQW15AN47NJ00D
- L3: renamed from L2; value 33n -> 47n; footprint (none) -> Inductor_SMD:L_0402_1005Metric_Pad0.77x0.64mm_HandSolder; MFR PART # (none) -> LQW15AN47NJ00D
- R49: renamed from R25; value 499R -> 470; footprint (none) -> Resistor_SMD:R_0805_2012Metric; LCSC (none) -> C17710
- R50: renamed from R24; footprint (none) -> Resistor_SMD:R_0402_1005Metric_Pad0.72x0.64mm_HandSolder; LCSC (none) -> C17168
- R51: renamed from R27; value 499R -> 470; footprint (none) -> Resistor_SMD:R_0805_2012Metric; LCSC (none) -> C17710
- R52: renamed from R32; value 49.9R -> 49.9; footprint (none) -> Resistor_SMD:R_0805_2012Metric; LCSC (none) -> C17720
- R53: renamed from R31; footprint (none) -> Resistor_SMD:R_1206_3216Metric; LCSC (none) -> C4410
- R54: renamed from R30; footprint (none) -> Resistor_SMD:R_0402_1005Metric_Pad0.72x0.64mm_HandSolder; LCSC (none) -> C17168
- R56: renamed from R28; value 499R -> 470; footprint (none) -> Resistor_SMD:R_0805_2012Metric; LCSC (none) -> C17710
- R57: renamed from R26; footprint (none) -> Resistor_SMD:R_0402_1005Metric_Pad0.72x0.64mm_HandSolder; LCSC (none) -> C17168
- R58: renamed from R29; value 499R -> 470; footprint (none) -> Resistor_SMD:R_0805_2012Metric; LCSC (none) -> C17710
- U3, U4, U5: MFR PART # (none) -> THS4631DR
Connections:
- net GND: now also R55.2
- net at C67.1, C71.1, R54.2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: now also R55.1
