File: hw/differential_probe/attenuators.kicad_sch (KiCad schematic)
At the start: 79 parts

Commit message: initial routing
Parts:
- removed C28: 470p, symbol Device:C
- removed C32: 5p, symbol Device:C
- removed R48: 0, symbol Device:R
- removed R49: 1M 0.1%, symbol Device:R
- added C33, C43: 4.7n, Capacitor_SMD:C_0805_2012Metric_Pad1.18x1.45mm_HandSolder, symbol Device:C
- added C34, C44: 220p, Capacitor_SMD:C_0805_2012Metric_Pad1.18x1.45mm_HandSolder, symbol Device:C
- added C35, C45: 47p, Capacitor_SMD:C_0805_2012Metric_Pad1.18x1.45mm_HandSolder, symbol Device:C
- added C37, C38, C39, C41: 10p, Capacitor_SMD:C_0805_2012Metric, symbol Device:C
- added R22: 0R, Resistor_SMD:R_1206_3216Metric_Pad1.30x1.75mm_HandSolder, symbol Device:R
- added R26, R27, R30: 1M 0.1%, Resistor_SMD:R_1206_3216Metric_Pad1.30x1.75mm_HandSolder, symbol Device:R
- 2M1: footprint (none) -> Potentiometer_THT:Potentiometer_Bourns_3296W_Vertical; MFR PART # (none) -> 3296W-1-500LF
- 2M2: value 50R -> 2M; footprint (none) -> Potentiometer_THT:Potentiometer_Bourns_3296W_Vertical; MFR PART # (none) -> 3296W-1-205LF
- C20: renamed from C60; value 10p -> 10p 6kV; footprint (none) -> Capacitor_THT:C_Rect_L9.0mm_W6.4mm_P7.50mm_MKT; MFR PART # (none) -> CC45SL3JD100JYVNA
- C21: renamed from C61; value 10p -> 10p 6kV; footprint (none) -> Capacitor_THT:C_Rect_L9.0mm_W6.4mm_P7.50mm_MKT; MFR PART # (none) -> CC45SL3JD100JYVNA
- C22: renamed from C62; value 10p -> 10p 6kV; footprint (none) -> Capacitor_THT:C_Rect_L9.0mm_W6.4mm_P7.50mm_MKT; MFR PART # (none) -> CC45SL3JD100JYVNA
- C23: renamed from C63; value 10p -> 10p 6kV; footprint (none) -> Capacitor_THT:C_Rect_L9.0mm_W6.4mm_P7.50mm_MKT; MFR PART # (none) -> CC45SL3JD100JYVNA
- C24: renamed from C64; value 10p -> 10p 6kV; footprint (none) -> Capacitor_THT:C_Rect_L9.0mm_W6.4mm_P7.50mm_MKT; MFR PART # (none) -> CC45SL3JD100JYVNA
- C25: renamed from C16; value 10p -> 10p 1kV; footprint (none) -> Capacitor_SMD:C_1206_3216Metric_Pad1.33x1.80mm_HandSolder; MFR PART # (none) -> SH31N100J102CT
- C26: renamed from C17; value 10p -> 10p 1kV; footprint (none) -> Capacitor_SMD:C_1206_3216Metric_Pad1.33x1.80mm_HandSolder; MFR PART # (none) -> SH31N100J102CT
- C27: renamed from C18; value 10p -> 10p 1kV; footprint (none) -> Capacitor_SMD:C_1206_3216Metric_Pad1.33x1.80mm_HandSolder; MFR PART # (none) -> SH31N100J102CT
- C28: renamed from C19; value 10p -> 10p 1kV; footprint (none) -> Capacitor_SMD:C_1206_3216Metric_Pad1.33x1.80mm_HandSolder; MFR PART # (none) -> SH31N100J102CT
- C29: renamed from C20; value 10p -> 10p 1kV; footprint (none) -> Capacitor_SMD:C_1206_3216Metric_Pad1.33x1.80mm_HandSolder; MFR PART # (none) -> SH31N100J102CT
- C30: renamed from C27; value 8~50p -> 8~28.5p; footprint (none) -> Capacitor_SMD:C_Trimmer_Voltronics_JZ; LCSC (none) -> C22468123
- C31: value 470p -> 10p; footprint (none) -> Capacitor_SMD:C_0805_2012Metric; LCSC (none) -> C1743
- C32: renamed from C30; footprint (none) -> Capacitor_SMD:C_0805_2012Metric; LCSC (none) -> C1743
- C36: renamed from C33; value 5p -> 10p; footprint (none) -> Capacitor_SMD:C_0805_2012Metric; LCSC (none) -> C1743
- C40: renamed from C26; value 8~50p -> 8~28.5p; footprint (none) -> Capacitor_SMD:C_Trimmer_Voltronics_JZ; LCSC (none) -> C22468123
- C42: renamed from C29; footprint (none) -> Capacitor_SMD:C_0805_2012Metric; LCSC (none) -> C1743
- C46: renamed from C21; value 10p -> 10p 1kV; footprint (none) -> Capacitor_SMD:C_1206_3216Metric_Pad1.33x1.80mm_HandSolder; MFR PART # (none) -> SH31N100J102CT
- C47: renamed from C22; value 10p -> 10p 1kV; footprint (none) -> Capacitor_SMD:C_1206_3216Metric_Pad1.33x1.80mm_HandSolder; MFR PART # (none) -> SH31N100J102CT
- C48: renamed from C23; value 10p -> 10p 1kV; footprint (none) -> Capacitor_SMD:C_1206_3216Metric_Pad1.33x1.80mm_HandSolder; MFR PART # (none) -> SH31N100J102CT
- C49: renamed from C24; value 10p -> 10p 1kV; footprint (none) -> Capacitor_SMD:C_1206_3216Metric_Pad1.33x1.80mm_HandSolder; MFR PART # (none) -> SH31N100J102CT
- C50: renamed from C25; value 10p -> 10p 1kV; footprint (none) -> Capacitor_SMD:C_1206_3216Metric_Pad1.33x1.80mm_HandSolder; MFR PART # (none) -> SH31N100J102CT
- C51: renamed from C39; value 10p -> 10p 6kV; footprint (none) -> Capacitor_THT:C_Rect_L9.0mm_W6.4mm_P7.50mm_MKT; MFR PART # (none) -> CC45SL3JD100JYVNA
- C52: renamed from C46; value 10p -> 10p 6kV; footprint (none) -> Capacitor_THT:C_Rect_L9.0mm_W6.4mm_P7.50mm_MKT; MFR PART # (none) -> CC45SL3JD100JYVNA
- C53: renamed from C57; value 10p -> 10p 6kV; footprint (none) -> Capacitor_THT:C_Rect_L9.0mm_W6.4mm_P7.50mm_MKT; MFR PART # (none) -> CC45SL3JD100JYVNA
- C54: renamed from C58; value 10p -> 10p 6kV; footprint (none) -> Capacitor_THT:C_Rect_L9.0mm_W6.4mm_P7.50mm_MKT; MFR PART # (none) -> CC45SL3JD100JYVNA
- C55: renamed from C59; value 10p -> 10p 6kV; footprint (none) -> Capacitor_THT:C_Rect_L9.0mm_W6.4mm_P7.50mm_MKT; MFR PART # (none) -> CC45SL3JD100JYVNA
- D6: renamed from D7; MFR PART # (none) -> BAS316
- D7: renamed from D6; MFR PART # (none) -> BAS316
- D8: renamed from D4; MFR PART # (none) -> BAS316
- D9: renamed from D5; MFR PART # (none) -> BAS316
- R10: renamed from R41; footprint (none) -> Resistor_THT:R_Axial_DIN0207_L6.3mm_D2.5mm_P10.16mm_Horizontal; MFR PART # (none) -> SM102031007FE
- R11: renamed from R42; footprint (none) -> Resistor_THT:R_Axial_DIN0207_L6.3mm_D2.5mm_P10.16mm_Horizontal; MFR PART # (none) -> SM102031007FE
- R12: renamed from R43; footprint (none) -> Resistor_THT:R_Axial_DIN0207_L6.3mm_D2.5mm_P10.16mm_Horizontal; MFR PART # (none) -> SM102031007FE
- R13: renamed from R44; footprint (none) -> Resistor_SMD:R_0805_2012Metric
- R14: renamed from R4; value 1M 0.1% -> 1M; footprint (none) -> Resistor_SMD:R_1206_3216Metric_Pad1.30x1.75mm_HandSolder; MFR PART # (none) -> CHV1206-FX-1004EST
- R15: renamed from R5; value 1M 0.1% -> 1M; footprint (none) -> Resistor_SMD:R_1206_3216Metric_Pad1.30x1.75mm_HandSolder; MFR PART # (none) -> CHV1206-FX-1004EST
- R16: renamed from R6; value 1M 0.1% -> 1M; footprint (none) -> Resistor_SMD:R_1206_3216Metric_Pad1.30x1.75mm_HandSolder; MFR PART # (none) -> CHV1206-FX-1004EST
- R17: renamed from R7; value 1M 0.1% -> 1M; footprint (none) -> Resistor_SMD:R_1206_3216Metric_Pad1.30x1.75mm_HandSolder; MFR PART # (none) -> CHV1206-FX-1004EST
- R18: renamed from R8; value 1M 0.1% -> 1M; footprint (none) -> Resistor_SMD:R_1206_3216Metric_Pad1.30x1.75mm_HandSolder; MFR PART # (none) -> CHV1206-FX-1004EST
- R19: renamed from R18; footprint (none) -> Resistor_SMD:R_1206_3216Metric_Pad1.30x1.75mm_HandSolder; LCSC (none) -> C17901
- R20: renamed from R23; footprint (none) -> Resistor_SMD:R_1206_3216Metric_Pad1.30x1.75mm_HandSolder; LCSC (none) -> C17901
- R21: renamed from R46; value 0 -> 0R; footprint (none) -> Resistor_SMD:R_1206_3216Metric_Pad1.30x1.75mm_HandSolder; LCSC (none) -> C17888
- R23: renamed from R16; footprint (none) -> Resistor_SMD:R_0603_1608Metric; LCSC (none) -> C22809
- R24: renamed from R22; footprint (none) -> Resistor_SMD:R_0603_1608Metric; LCSC (none) -> C22809
- R25: renamed from R17; value 10k 0.1% -> 20k 0.1%; footprint (none) -> Resistor_SMD:R_1206_3216Metric_Pad1.30x1.75mm_HandSolder; MFR PART # (none) -> RNCF1206BTE20K0
- R28: renamed from R15; value 10k 0.1% -> 20k 0.1%; footprint (none) -> Resistor_SMD:R_1206_3216Metric_Pad1.30x1.75mm_HandSolder; MFR PART # (none) -> RNCF1206BTE20K0
- R29: renamed from R50; footprint (none) -> Resistor_SMD:R_1206_3216Metric_Pad1.30x1.75mm_HandSolder; MFR PART # (none) -> RNCS1206BKE1M00
- R31: renamed from R20; footprint (none) -> Resistor_SMD:R_0603_1608Metric; LCSC (none) -> C22809
- R32: renamed from R21; footprint (none) -> Resistor_SMD:R_0603_1608Metric; LCSC (none) -> C22809
- R33: renamed from R45; value 10R -> 118R; footprint (none) -> Resistor_SMD:R_1206_3216Metric_Pad1.30x1.75mm_HandSolder; MFR PART # (none) -> RMCF1206FT118R
- R34: renamed from R51; value 100k -> 470k; footprint (none) -> Resistor_SMD:R_0805_2012Metric; MFR PART # (none) -> C17709; now fitted
- R35: renamed from R52; value 10M -> 10M 0.1%; footprint (none) -> Resistor_SMD:R_1206_3216Metric_Pad1.30x1.75mm_HandSolder; MFR PART # (none) -> MCA1206MD1005BP100
- R36: renamed from R9; value 1M 0.1% -> 1M; footprint (none) -> Resistor_SMD:R_1206_3216Metric_Pad1.30x1.75mm_HandSolder; MFR PART # (none) -> CHV1206-FX-1004EST
- R37: renamed from R10; value 1M 0.1% -> 1M; footprint (none) -> Resistor_SMD:R_1206_3216Metric_Pad1.30x1.75mm_HandSolder; MFR PART # (none) -> CHV1206-FX-1004EST
- R38: renamed from R11; value 1M 0.1% -> 1M; footprint (none) -> Resistor_SMD:R_1206_3216Metric_Pad1.30x1.75mm_HandSolder; MFR PART # (none) -> CHV1206-FX-1004EST
- R39: renamed from R12; value 1M 0.1% -> 1M; footprint (none) -> Resistor_SMD:R_1206_3216Metric_Pad1.30x1.75mm_HandSolder; MFR PART # (none) -> CHV1206-FX-1004EST
- R40: renamed from R13; value 1M 0.1% -> 1M; footprint (none) -> Resistor_SMD:R_1206_3216Metric_Pad1.30x1.75mm_HandSolder; MFR PART # (none) -> CHV1206-FX-1004EST
- R41: renamed from R14; footprint (none) -> Resistor_SMD:R_1206_3216Metric_Pad1.30x1.75mm_HandSolder; LCSC (none) -> C17901
- R42: renamed from R19; footprint (none) -> Resistor_SMD:R_1206_3216Metric_Pad1.30x1.75mm_HandSolder; LCSC (none) -> C17901
- R43: renamed from R38; footprint (none) -> Resistor_SMD:R_0805_2012Metric
- R44: renamed from R33; footprint (none) -> Resistor_THT:R_Axial_DIN0207_L6.3mm_D2.5mm_P10.16mm_Horizontal; MFR PART # (none) -> SM102031007FE
- R45: renamed from R34; footprint (none) -> Resistor_THT:R_Axial_DIN0207_L6.3mm_D2.5mm_P10.16mm_Horizontal; MFR PART # (none) -> SM102031007FE
- R46: renamed from R35; footprint (none) -> Resistor_THT:R_Axial_DIN0207_L6.3mm_D2.5mm_P10.16mm_Horizontal; MFR PART # (none) -> SM102031007FE
- R47: renamed from R36; footprint (none) -> Resistor_THT:R_Axial_DIN0207_L6.3mm_D2.5mm_P10.16mm_Horizontal; MFR PART # (none) -> SM102031007FE
- R48: renamed from R37; footprint (none) -> Resistor_THT:R_Axial_DIN0207_L6.3mm_D2.5mm_P10.16mm_Horizontal; MFR PART # (none) -> SM102031007FE
- R8: renamed from R39; footprint (none) -> Resistor_THT:R_Axial_DIN0207_L6.3mm_D2.5mm_P10.16mm_Horizontal; MFR PART # (none) -> SM102031007FE
- R9: renamed from R40; footprint (none) -> Resistor_THT:R_Axial_DIN0207_L6.3mm_D2.5mm_P10.16mm_Horizontal; MFR PART # (none) -> SM102031007FE
- RV1: renamed from RV2; footprint (none) -> Potentiometer_THT:Potentiometer_Bourns_3296Y_Vertical; MFR PART # (none) -> 3296Y-1-105LF
- RV2: renamed from RV3; footprint (none) -> Potentiometer_THT:Potentiometer_Bourns_3296Y_Vertical; MFR PART # (none) -> 3296Y-1-105LF
- TP1: renamed from TP4; footprint (none) -> TestPoint:TestPoint_Loop_D2.50mm_Drill1.85mm
- TP2: renamed from TP1; footprint (none) -> TestPoint:TestPoint_Loop_D2.50mm_Drill1.85mm
- TP3: renamed from TP2; footprint (none) -> TestPoint:TestPoint_Loop_D2.50mm_Drill1.85mm
- TP4: renamed from TP3; footprint (none) -> TestPoint:TestPoint_Loop_D2.50mm_Drill1.85mm
Connections:
- net ATTEN-: now also C39.1
- net GND: now also C33.1, C34.1, C35.1, C37.2, C38.2, C41.1, C43.1, C44.1, C45.1; no longer C36.2
- net at C40.2, C42.2, D8.2 (A)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: now also C41.2, C43.2, C44.2, C45.2
- net at C30.2, C31.2, C32.2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: now also C33.2, C34.2, C35.2, R22.2
- net at 2M1.1, 2M2.2, R28.1: now also R30.1; no longer R29.1
- net at 2M1.3, R25.1: now also R27.1
- new net: C36.2, C37.1
- new net: R22.1, R26.2
- new net: R26.1, R27.2
- new net: R29.1, R30.2
- new net: C38.1, C39.2
Other:
- note added: "LV 1:250 Attenuation 5M, 2pF Impedance ±2.5kV -> ±10V HV 1:2500 Attenuation 5G, 2pF Impedance ±25kV -> ±10V"
- note added: "OHMITE 1G 5.0kV SM102031007FE TDK 10pF 6.0kV CC45SL3JD100JYVNA BROUNS 1M 3.0kV CHV1206-FX-1004EST WALSIN 10p 1kV SH31N100J102CT"
- note removed: "1:500 Attenuation 5M, 2pF Impedance"
- note removed: "OHMITE 1G 5.0kV SM102031007FE TDK 10pF 6.0kV CC45SL3JD100JYVNA"
- moved on the sheet: 2M1, 2M2, C20, C21, C22, C23, C24, C25, C26, C27, C28, C29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
