File: hw/differential_probe/differential_probe.kicad_sch (KiCad schematic)
At the start: 1 part, among them J1 IPX

Commit message: initial routing
Parts:
- added J1: RFShield_OnePiece, symbol Device:RFShield_OnePiece
- J2: renamed from J1; MFR PART # (none) -> C496552
Connections:
- net GND: now also J1.1 (Shield)
Other:
- moved on the sheet: J2
