File: hw/differential_probe/power.kicad_sch (KiCad schematic)
At the start: 32 parts, among them P1 USB_C_Plug_USB2.0, T1 1006_760390014, U1 SN6505BDBV, U6 L78L15_SOT89, U7 L79L15_SOT89

Commit message: initial routing
Parts:
- removed C4, C5: 100n, symbol Device:C
- removed C6: 10u, symbol Device:C
- removed D3: LED, symbol Device:LED
- removed P1: USB_C_Plug_USB2.0, symbol Connector:USB_C_Plug_USB2.0
- removed U6: L78L15_SOT89, Package_TO_SOT_SMD:SOT-89-3, symbol Regulator_Linear:L78L15_SOT89
- removed U7: L79L15_SOT89, Package_TO_SOT_SMD:SOT-89-3, symbol Regulator_Linear:L79L15_SOT89
- added C16, C18: 10u, Capacitor_SMD:C_1206_3216Metric, symbol Device:C
- added C17: 100n, Capacitor_SMD:C_0402_1005Metric, symbol Device:C
- added C19: 10n, Capacitor_SMD:C_0805_2012Metric, symbol Device:C
- added D5: LED, LED_SMD:LED_0805_2012Metric, symbol Device:LED
- added H1: Light Guide, Bivar_SLP3_Light_Pipe:SLP3-150-100-F, symbol Mechanical:MountingHole
- added J3: USB_C_Receptacle_USB2.0_16P, G_SWITCH_USB-C:USB_C_Receptacle_G-Switch_GT-USB-7043, symbol Connector:USB_C_Receptacle_USB2.0_16P
- added L1: 1812_744235510, WE Chokes:L_Wurth_WE-CNSW-1812, symbol WE chokes:1812_744235510
- added R2: 33k, Resistor_SMD:R_0805_2012Metric, symbol Device:R
- added R4: 115k, Resistor_SMD:R_0402_1005Metric_Pad0.72x0.64mm_HandSolder, symbol Device:R
- added R5: 0R, Resistor_SMD:R_0402_1005Metric_Pad0.72x0.64mm_HandSolder, symbol Device:R
- added R6: 10k, Resistor_SMD:R_0402_1005Metric, symbol Device:R
- added R7: 127k, Resistor_SMD:R_0402_1005Metric_Pad0.72x0.64mm_HandSolder, symbol Device:R
- added U2: TPS7A39, Package_SON:Texas_S-PVSON-N10_ThermalVias, symbol Regulator_Linear:TPS7A39
- C1: renamed from C2; footprint (none) -> Capacitor_SMD:C_1206_3216Metric; LCSC (none) -> C13585
- C10, C12: footprint (none) -> Capacitor_SMD:C_0402_1005Metric; LCSC (none) -> C307331
- C11, C14: value 100n -> 10u; footprint (none) -> Capacitor_SMD:C_1206_3216Metric; LCSC (none) -> C13585
- C13, C15, C8: value 10u -> 100n; footprint (none) -> Capacitor_SMD:C_0402_1005Metric; LCSC (none) -> C307331
- C2: renamed from C3; footprint (none) -> Capacitor_SMD:C_0402_1005Metric; LCSC (none) -> C307331
- C3: renamed from C55; footprint (none) -> Capacitor_SMD:C_1206_3216Metric; LCSC (none) -> C13585
- C4: renamed from C56; footprint (none) -> Capacitor_SMD:C_0402_1005Metric; LCSC (none) -> C307331
- C5: renamed from C53; footprint (none) -> Capacitor_SMD:C_1206_3216Metric; LCSC (none) -> C13585
- C6: renamed from C54; footprint (none) -> Capacitor_SMD:C_0402_1005Metric; LCSC (none) -> C307331
- C7, C9: footprint (none) -> Capacitor_SMD:C_1206_3216Metric; LCSC (none) -> C13585
- D1: renamed from D8; value MBR0530 -> MBR0530T1G; MFR PART # (none) -> MBR0530T1G
- D2: footprint (none) -> LED_SMD:LED_0805_2012Metric; LCSC (none) -> C34499
- D3: renamed from D1; footprint (none) -> Diode_SMD:D_SMA_Handsoldering; MFR PART # (none) -> SMAJ6.5A
- D4: renamed from D9; value MBR0530 -> MBR0530T1G; MFR PART # (none) -> MBR0530T1G
- FB1, FB2: footprint (none) -> Inductor_SMD:L_0402_1005Metric_Pad0.77x0.64mm_HandSolder; MFR PART # (none) -> LQW15AN47NJ00D
- R1: renamed from R2; value 4k7 -> 33k; footprint (none) -> Resistor_SMD:R_0805_2012Metric; LCSC (none) -> C17633
- R3: value 4k7 -> 10k; footprint (none) -> Resistor_SMD:R_0402_1005Metric; LCSC (none) -> C25744
- T1: footprint Transformer_SMD_Wurth:T_Wurth_WE-PPTI-1006 -> WE Inductor:T_Wurth_WE-PPTI-1006; MFR PART # (none) -> 760390014
- U1: LCSC (none) -> C74518
Connections:
- net +15V: now also C10.1, C11.1, L1.3; no longer C12.1, C13.1, FB1.2
- net +24V: now also C7.1, C8.1, R1.2, R5.1, U2.1 (INP)
- net -15V: now also C17.2, C18.2, L1.2; no longer C14.2, C15.2, FB2.2
- net -24V: now also C14.2, C15.2, D5.1 (K), U2.5 (INN); no longer C7.2
- net GND: now also C11.2, C7.2, C9.2, R3.1, C16.1, C17.1, C18.1, C19.2, R2.2, U2.11 (GND), U2.4 (GND); no longer C11.1, C12.2, C13.2, C7.1, C9.1, R3.2
- net GNDPWR: now also J3.A1 (GND), J3.A12 (GND), J3.B1 (GND), J3.B12 (GND), J3.S1 (SHIELD)
- net at C1.1, C2.1, D3.1 (K)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: now also J3.A4 (VBUS), J3.A9 (VBUS), J3.B4 (VBUS), J3.B9 (VBUS)
- net at U1.1 (D1): now also T1.3; no longer T1.1
- net at U1.3 (D2): now also T1.1; no longer T1.3
- new net: C13.1, C16.2, FB2.1, R7.1, U2.6 (OUTN)
- new net: D5.2 (A), R2.1
- new net: R6.1, U2.8 (BUF)
- new net: C13.2, R6.2, R7.2, U2.7 (FBN)
- new net: FB2.2, L1.1
- new net: FB1.2, L1.4
- new net: C19.1, U2.3 (NR/SS)
- new net: C12.1, C9.1, FB1.1, R4.2, U2.10 (OUTP)
- new net: R5.2, U2.2 (EN)
- new net: C12.2, R3.2, R4.1, U2.9 (FBP)
- no-connect marks 5 -> 9
Other:
- moved on the sheet: C1, C2, C3, C4, C5, C6, D1, D2, D3, D4, R1, T1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
